Commit message: amcl base_link warning

File: my_robot/urdf/my_robot.xacro (robot description, xacro)
@@ -3,5 +3,6 @@
   <xacro:include filename="$(find my_robot)/urdf/my_robot.gazebo" />
   <!-- Import gazebo elements -->
-  <link name="robot_footprint" />
+  <!-- <link name="robot_footprint" /> --> <!-- nov05 -->
+  <link name="base_link" />                <!-- nov05 -->
   <link name='chassis'>
     <pose>0 0 0.1 0 0 0</pose>

Commit message: .

File: my_robot/urdf/my_robot.xacro (robot description, xacro)
@@ -52,7 +52,9 @@
     </visual>
   </link>
-  <joint name="robot_footprint_joint" type="fixed">
+  <!-- <joint name="robot_footprint_joint" type="fixed"> --> <!-- nov05 -->
+  <joint name="base_link_joint" type="fixed">                <!-- nov05 -->
     <origin xyz="0 0 0" rpy="0 0 0" />
-    <parent link="robot_footprint" />
+    <!-- <parent link="robot_footprint" /> -->               <!-- nov05 -->
+    <parent link="base_link" />                              <!-- nov05 -->
     <child link="chassis" />
   </joint>

Commit message: .

File: my_robot/urdf/my_robot.xacro (robot description, xacro)
@@ -85,5 +85,6 @@
     <origin xyz="0 0.15 0" rpy="0 0 0" />
     <child link="left_wheel" />
-    <parent link="chassis" />
+    <!-- <parent link="chassis" /> --> <!-- nov05 -->
+    <parent link="base_link" />        <!-- nov05 -->
     <axis xyz="0 1 0" rpy="0 0 0" />
     <limit effort="10000" velocity="1000" />
@@ -115,5 +116,6 @@
     <origin xyz="0 -0.15 0" rpy="0 0 0" />
     <child link="right_wheel" />
-    <parent link="chassis" />
+    <!-- <parent link="chassis" /> -->  <!-- nov05 -->
+    <parent link="base_link" />         <!-- nov05 -->
     <axis xyz="0 1 0" rpy="0 0 0" />
     <limit effort="10000" velocity="1000" />

Commit message: change my_robot urdf, base_link related

File: my_robot/urdf/my_robot.xacro (robot description, xacro)
@@ -85,6 +85,5 @@
     <origin xyz="0 0.15 0" rpy="0 0 0" />
     <child link="left_wheel" />
-    <!-- <parent link="chassis" /> --> <!-- nov05 -->
-    <parent link="base_link" />        <!-- nov05 -->
+    <parent link="chassis" />
     <axis xyz="0 1 0" rpy="0 0 0" />
     <limit effort="10000" velocity="1000" />
@@ -116,6 +115,5 @@
     <origin xyz="0 -0.15 0" rpy="0 0 0" />
     <child link="right_wheel" />
-    <!-- <parent link="chassis" /> -->  <!-- nov05 -->
-    <parent link="base_link" />         <!-- nov05 -->
+    <parent link="chassis" />
     <axis xyz="0 1 0" rpy="0 0 0" />
     <limit effort="10000" velocity="1000" />
